File: Pushpull-Highside-Driver/Pushpull-Highside-Driver.kicad_sch (KiCad schematic)
At the start: 17 parts, among them J1 Last, J2 Controller-IO, J3 24V Versorgung, Q1 BC846, Q2 BC846, Q3 BC856, Q4 IRFR120N

Commit message: Footprint
Parts:
- C1, C2, C3: footprint (none) -> Capacitor_SMD:C_0805_2012Metric_Pad1.18x1.45mm_HandSolder
- D1: footprint (none) -> Diode_SMD:D_MiniMELF_Handsoldering
- R1, R2, R3, R4, R5: footprint (none) -> PCM_Resistor_SMD_AKL:R_1206_3216Metric_Pad1.42x1.75mm_HandSolder
Changed lines of the file:
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@@
       (effects (font (size 1.27 1.27)))
     )
-    (property "Footprint" "" (at 160.02 86.868 90)
+    (property "Footprint" "PCM_Resistor_SMD_AKL:R_1206_3216Metric_Pad1.42x1.75mm_HandSolder" (at 160.02 86.868 90)
       (effects (font (size 1.27 1.27)) hide)
     )
@@
       (effects (font (size 1.27 1.27)))
     )
-    (property "Footprint" "" (at 110.49 132.588 90)
+    (property "Footprint" "PCM_Resistor_SMD_AKL:R_1206_3216Metric_Pad1.42x1.75mm_HandSolder" (at 110.49 132.588 90)
       (effects (font (size 1.27 1.27)) hide)
     )
@@
       (effects (font (size 1.27 1.27)) (justify left))
     )
-    (property "Footprint" "" (at 104.902 53.34 90)
+    (property "Footprint" "PCM_Resistor_SMD_AKL:R_1206_3216Metric_Pad1.42x1.75mm_HandSolder" (at 104.902 53.34 90)
       (effects (font (size 1.27 1.27)) hide)
     )
@@
       (effects (font (size 1.27 1.27)) (justify left))
     )
-    (property "Footprint" "" (at 93.98 68.58 0)
+    (property "Footprint" "Diode_SMD:D_MiniMELF_Handsoldering" (at 93.98 68.58 0)
       (effects (font (size 1.27 1.27)) hide)
     )
@@
       (effects (font (size 1.27 1.27)) (justify left))
     )
-    (property "Footprint" "" (at 130.302 69.85 90)
+    (property "Footprint" "PCM_Resistor_SMD_AKL:R_1206_3216Metric_Pad1.42x1.75mm_HandSolder" (at 130.302 69.85 90)
       (effects (font (size 1.27 1.27)) hide)
     )
@@
       (effects (font (size 1.27 1.27)) (justify right))
     )
-    (property "Footprint" "" (at 133.858 149.86 90)
+    (property "Footprint" "PCM_Resistor_SMD_AKL:R_1206_3216Metric_Pad1.42x1.75mm_HandSolder" (at 133.858 149.86 90)
       (effects (font (size 1.27 1.27)) hide)
     )
@@
       (effects (font (size 1.27 1.27)) (justify left))
     )
-    (property "Footprint" "" (at 107.6452 72.39 0)
+    (property "Footprint" "Capacitor_SMD:C_0805_2012Metric_Pad1.18x1.45mm_HandSolder" (at 107.6452 72.39 0)
       (effects (font (size 1.27 1.27)) hide)
     )
@@
       (effects (font (size 1.27 1.27)))
     )
-    (property "Footprint" "" (at 114.3 118.4148 0)
+    (property "Footprint" "Capacitor_SMD:C_0805_2012Metric_Pad1.18x1.45mm_HandSolder" (at 114.3 118.4148 0)
       (effects (font (size 1.27 1.27)) hide)
     )
@@
       (effects (font (size 1.27 1.27)) (justify left))
     )
-    (property "Footprint" "" (at 124.1552 87.63 0)
-      (effects (font (size 1.27 1.27)) hide)
-    )
+    (property "Footprint" "Capacitor_SMD:C_0805_2012Metric_Pad1.18x1.45mm_HandSolder" (at 124.1552 87.63 0)
+      (effects (font (size 1.27 1.27)) hide)
+    )

Commit message: PCB added
Parts:
- D2: footprint Diode_SMD_AKL:D_MiniMELF -> PCM_Diode_SMD_AKL:D_MiniMELF_Handsoldering
- Q1, Q2, Q3: footprint Package_TO_SOT_SMD_AKL:SOT-23 -> PCM_Package_TO_SOT_SMD_AKL:SOT-23
- Q4: footprint Package_TO_SOT_SMD_AKL:TO-252-2 -> PCM_Package_TO_SOT_SMD_AKL:TO-252-2
Changed lines of the file:
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@@
       (effects (font (size 1.27 1.27)) (justify left))
     )
-    (property "Footprint" "Package_TO_SOT_SMD_AKL:TO-252-2" (at 180.34 81.28 0)
+    (property "Footprint" "PCM_Package_TO_SOT_SMD_AKL:TO-252-2" (at 180.34 81.28 0)
       (effects (font (size 1.27 1.27)) hide)
     )
@@
       (effects (font (size 1.27 1.27)))
     )
-    (property "Footprint" "Diode_SMD_AKL:D_MiniMELF" (at 114.3 63.5 0)
+    (property "Footprint" "PCM_Diode_SMD_AKL:D_MiniMELF_Handsoldering" (at 114.3 63.5 0)
       (effects (font (size 1.27 1.27)) hide)
     )
@@
       (effects (font (size 1.27 1.27)) (justify left))
     )
-    (property "Footprint" "Package_TO_SOT_SMD_AKL:SOT-23" (at 149.86 92.71 0)
+    (property "Footprint" "PCM_Package_TO_SOT_SMD_AKL:SOT-23" (at 149.86 92.71 0)
       (effects (font (size 1.27 1.27)) hide)
     )
@@
       (effects (font (size 1.27 1.27)) (justify left))
     )
-    (property "Footprint" "Package_TO_SOT_SMD_AKL:SOT-23" (at 134.62 128.27 0)
+    (property "Footprint" "PCM_Package_TO_SOT_SMD_AKL:SOT-23" (at 134.62 128.27 0)
       (effects (font (size 1.27 1.27)) hide)
     )
@@
       (effects (font (size 1.27 1.27)) (justify left))
     )
-    (property "Footprint" "Package_TO_SOT_SMD_AKL:SOT-23" (at 149.86 73.66 0)
-      (effects (font (size 1.27 1.27)) hide)
-    )
+    (property "Footprint" "PCM_Package_TO_SOT_SMD_AKL:SOT-23" (at 149.86 73.66 0)
+      (effects (font (size 1.27 1.27)) hide)
+    )
